File: HandwireCustom.kicad_pcb (KiCad board)
At the start: 2 copper layers, 285.8 x 121.4 mm, 148 parts, among them J1 ICSP, J2 Conn_01x04, K0 KEYSW, K1 KEYSW, K10 KEYSW, K11 KEYSW, K110 KEYSW, K111 KEYSW, K112 KEYSW, K113 KEYSW, K12 KEYSW, K13 KEYSW, K14 KEYSW, K15 KEYSW, K16 KEYSW, K17 KEYSW, K18 KEYSW, K19 KEYSW, K2 KEYSW, K20 KEYSW, K21 KEYSW, K210 KEYSW, K211 KEYSW, K213 KEYSW, K22 KEYSW, K23 KEYSW, K24 KEYSW, K25 KEYSW, K26 KEYSW, K27 KEYSW, K28 KEYSW, K29 KEYSW, K3 KEYSW, K30 KEYSW, K31 KEYSW, K310 KEYSW, K311 KEYSW, K313 KEYSW, K32 KEYSW, K33 KEYSW, K34 KEYSW, K35 KEYSW, K36 KEYSW, K37 KEYSW, K38 KEYSW, K39 KEYSW, K4 KEYSW, K40 KEYSW, K41 KEYSW, K410 KEYSW, K411 KEYSW, K413 KEYSW, K42 KEYSW, K45 KEYSW, K48 KEYSW, K49 KEYSW, K5 KEYSW, K6 KEYSW, K7 KEYSW, K8 KEYSW, K9 KEYSW, SW1 SW_Push, U1 ATmega32U4RC-M, Y1 Crystal

Commit message: 2nd row done
Routing:
- net Net-(D5-Pad2): track 277.2 -> 0.00 mm, vias 9 -> 0
- net Net-(D10-Pad2): track 256.8 -> 0.00 mm, vias 9 -> 0
- net Col13: track 337.9 -> 86.1 mm, vias 7 -> 0
- net Net-(D15-Pad2): track 236.1 -> 0.00 mm, vias 7 -> 0
- net Col12: track 250.7 -> 23.3 mm, vias 5 -> 0
- net Col11: track 311.6 -> 96.2 mm, vias 9 -> 0
- net Net-(D4-Pad2): track 200.8 -> 0.00 mm, vias 3 -> 0
- net Col10: track 288.1 -> 92.3 mm, vias 9 -> 0
- net Col9: track 278.7 -> 92.0 mm, vias 5 -> 0
- net Net-(D9-Pad2): track 173.6 -> 0.00 mm, vias 3 -> 0
- net Col8: track 258.0 -> 92.0 mm, vias 7 -> 0
- net Net-(D14-Pad2): track 155.8 -> 0.00 mm, vias 3 -> 0
- net Net-(D28-Pad2): track 156.8 -> 2.15 mm, vias 5 -> 1
- net Net-(D61-Pad2): track 154.0 -> 0.00 mm, vias 1 -> 0
- net Net-(D3-Pad2): track 149.6 -> 0.00 mm, vias 1 -> 0
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
Commit message: Completed
DRC: 0 Errors, 0 Warnings
Parts:
- removed K311, K411: KEYSW, MX_Only:MXOnly-1U-Hotswap
- added K312: KEYSW, MX_Only:MXOnly-1U-Hotswap, F.Cu at (325.4, 177.0)
- added K412: KEYSW, MX_Only:MXOnly-1U-Hotswap, F.Cu at (325.4, 196.1)
Connections:
- U1 pad 26: Col13 -> Col2
- U1 pad 27: Col12 -> Col3
- U1 pad 28: Col11 -> Col4
- U1 pad 29: Col10 -> Col5
- U1 pad 30: Col9 -> Col6
- U1 pad 31: Col8 -> Col7
- U1 pad 32: Col7 -> Col8
- U1 pad 36: Col5 -> Col9
- U1 pad 37: Col4 -> Col10
- U1 pad 38: Col3 -> Col11
- U1 pad 39: Col2 -> Col12
- U1 pad 40: Col1 -> Col13
- U1 pad 8: unconnected-(U1-Pad8) -> Col1
Routing:
- net Col12: track 23.3 -> 417.3 mm, vias 0 -> 5
- net Col13: track 86.1 -> 436.7 mm, vias 0 -> 5
- net Col11: track 96.2 -> 429.1 mm, vias 0 -> 5
- net Col10: track 92.3 -> 406.4 mm, vias 0 -> 5
- net Net-(D5-Pad2): track 0.00 -> 306.4 mm, vias 0 -> 7
- net Col9: track 92.0 -> 386.0 mm, vias 0 -> 5
- net Net-(D10-Pad2): track 0.00 -> 280.9 mm, vias 0 -> 5
- net Col8: track 92.0 -> 362.3 mm, vias 0 -> 5
- net Net-(D15-Pad2): track 0.00 -> 256.9 mm, vias 0 -> 5
- net Net-(D4-Pad2): track 0.00 -> 227.4 mm, vias 0 -> 3
- net Net-(D9-Pad2): track 0.00 -> 198.5 mm, vias 0 -> 3
- net Net-(D28-Pad2): track 2.15 -> 189.9 mm, vias 1 -> 5
- net Net-(D14-Pad2): track 0.00 -> 181.2 mm, vias 0 -> 3
- net Net-(D3-Pad2): track 0.00 -> 169.9 mm, vias 0 -> 1
- net Net-(D61-Pad2): track 0.00 -> 164.9 mm, vias 0 -> 1
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