File: untitled.kicad_sch (KiCad schematic)
At the start: 126 parts, among them K0 KEYSW, K1 KEYSW, K10 KEYSW, K11 KEYSW, K110 KEYSW, K111 KEYSW, K112 KEYSW, K113 KEYSW, K12 KEYSW, K13 KEYSW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

Commit message: Completed
DRC: 0 Errors, 0 Warnings
Parts:
- renumbered K311 to K312, K411 to K412
Connections:
- net Col11: no longer K312.1, K412.1
- net Col12: now also K312.1, K412.1
Other:
- moved on the sheet: D55, D56, K312, K412
