File: HandwireCustom.kicad_sch (KiCad schematic)
At the start: 22 parts, among them J1 ICSP, J2 Conn_01x04, SW1 SW_Push, U1 ATmega32U4RC-M, Y1 Crystal

Commit message: Completed
DRC: 0 Errors, 0 Warnings
Connections:
- net Col0 is gone; now on net Col2: U1.12 (PB7)
- net Col1: now also U1.8 (PB0); no longer U1.40 (PF1)
- net Col10: now also U1.37 (PF6); no longer U1.29 (PB5)
- net Col11: now also U1.38 (PF5); no longer U1.28 (PB4)
- net Col12: now also U1.39 (PF4); no longer U1.27 (PD7)
- net Col13: now also U1.40 (PF1); no longer U1.26 (PD6)
- net Col2: now also U1.26 (PD6); no longer U1.39 (PF4)
- net Col3: now also U1.27 (PD7); no longer U1.38 (PF5)
- net Col4: now also U1.28 (PB4); no longer U1.37 (PF6)
- net Col5: now also U1.29 (PB5); no longer U1.36 (PF7)
- net Col7: now also U1.31 (PC6); no longer U1.32 (PC7)
- net Col8: now also U1.32 (PC7); no longer U1.31 (PC6)
- net Col9: now also U1.36 (PF7); no longer U1.30 (PB6)
- new net Col6: U1.30 (PB6)
- no-connect marks 5 -> 4
Changed lines of the file:
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@@
   )
   (no_connect (at 37.592 103.378))
-  (no_connect (at 124.714 38.1))
   (no_connect (at 124.714 93.98))
   (no_connect (at 37.592 118.618))
@@
     (stroke (width 0) (type default) (color 0 0 0 0))
   )
+  (wire (pts (xy 124.714 38.1) (xy 127.508 38.1))
+    (stroke (width 0) (type default) (color 0 0 0 0))
+  )
   (polyline (pts (xy 51.816 83.566) (xy 51.816 45.212))
     (stroke (width 0) (type default) (color 0 0 0 0))
@@
     )
   )
-  (global_label "Col9" (shape input) (at 127.508 53.34 0) (fields_autoplaced)
+  (global_label "Col6" (shape input) (at 127.508 53.34 0) (fields_autoplaced)
     (effects (font (size 1 1)) (justify left))
     (property "Intersheet References" "${INTERSHEET_REFS}" (id 0) (at 132.789 53.2775 0)
@@
     )
   )
-  (global_label "Col13" (shape input) (at 127.508 83.82 0) (fields_autoplaced)
-    (effects (font (size 1 1)) (justify left))
-    (property "Intersheet References" "${INTERSHEET_REFS}" (id 0) (at 133.7413 83.7575 0)
+  (global_label "Col2" (shape input) (at 127.508 83.82 0) (fields_autoplaced)
+    (effects (font (size 1 1)) (justify left))
+    (property "Intersheet References" "${INTERSHEET_REFS}" (id 0) (at 132.789 83.7575 0)
       (effects (font (size 1 1)) (justify left) hide)
     )
@@
     )
   )
-  (global_label "Col2" (shape input) (at 127.508 104.14 0) (fields_autoplaced)
-    (effects (font (size 1 1)) (justify left))
-    (property "Intersheet References" "${INTERSHEET_REFS}" (id 0) (at 132.789 104.0775 0)
+  (global_label "Col12" (shape input) (at 127.508 104.14 0) (fields_autoplaced)
+    (effects (font (size 1 1)) (justify left))
+    (property "Intersheet References" "${INTERSHEET_REFS}" (id 0) (at 133.7413 104.0775 0)
       (effects (font (size 1 1)) (justify left) hide)
     )
@@
     )
   )
-  (global_label "Col4" (shape input) (at 127.508 109.22 0) (fields_autoplaced)
-    (effects (font (size 1 1)) (justify left))
-    (property "Intersheet References" "${INTERSHEET_REFS}" (id 0) (at 132.789 109.1575 0)
+  (global_label "Col10" (shape input) (at 127.508 109.22 0) (fields_autoplaced)
+    (effects (font (size 1 1)) (justify left))
+    (property "Intersheet References" "${INTERSHEET_REFS}" (id 0) (at 133.7413 109.1575 0)
       (effects (font (size 1 1)) (justify left) hide)
     )
@@
     )
   )
-  (global_label "Col10" (shape input) (at 127.508 50.8 0) (fields_autoplaced)
-    (effects (font (size 1 1)) (justify left))
-    (property "Intersheet References" "${INTERSHEET_REFS}" (id 0) (at 133.7413 50.7375 0)
+  (global_label "Col5" (shape input) (at 127.508 50.8 0) (fields_autoplaced)
+    (effects (font (size 1 1)) (justify left))
+    (property "Intersheet References" "${INTERSHEET_REFS}" (id 0) (at 132.789 50.7375 0)
       (effects (font (size 1 1)) (justify left) hide)
     )
@@
     )
   )
-  (global_label "Col11" (shape input) (at 127.508 48.26 0) (fields_autoplaced)
-    (effects (font (size 1 1)) (justify left))
-    (property "Intersheet References" "${INTERSHEET_REFS}" (id 0) (at 133.7413 48.1975 0)
+  (global_label "Col4" (shape input) (at 127.508 48.26 0) (fields_autoplaced)
+    (effects (font (size 1 1)) (justify left))
+    (property "Intersheet References" "${INTERSHEET_REFS}" (id 0) (at 132.789 48.1975 0)
       (effects (font (size 1 1)) (justify left) hide)
     )
@@
     )
   )
-  (global_label "Col7" (shape input) (at 127.508 63.5 0) (fields_autoplaced)
+  (global_label "Col8" (shape input) (at 127.508 63.5 0) (fields_autoplaced)
     (effects (font (size 1 1)) (justify left))
     (property "Intersheet References" "${INTERSHEET_REFS}" (id 0) (at 132.789 63.4375 0)
@@
     )
   )
-  (global_label "Col12" (shape input) (at 127.508 86.36 0) (fields_autoplaced)
-    (effects (font (size 1 1)) (justify left))
-    (property "Intersheet References" "${INTERSHEET_REFS}" (id 0) (at 133.7413 86.2975 0)
-      (effects (font (size 1 1)) (justify left) hide)
-    )
-  )
-  (global_label "Col0" (shape input) (at 127.508 55.88 0) (fields_autoplaced)
+  (global_label "Col3" (shape input) (at 127.508 86.36 0) (fields_autoplaced)
+    (effects (font (size 1 1)) (justify left))
+    (property "Intersheet References" "${INTERSHEET_REFS}" (id 0) (at 132.789 86.2975 0)
+      (effects (font (size 1 1)) (justify left) hide)
+    )
+  )
+  (global_label "Col2" (shape input) (at 127.508 55.88 0) (fields_autoplaced)
     (effects (font (size 1 1)) (justify left))
     (property "Intersheet References" "${INTERSHEET_REFS}" (id 0) (at 132.789 55.8175 0)
@@
     )
   )
+  (global_label "Col1" (shape input) (at 127.508 38.1 0) (fields_autoplaced)
+    (effects (font (size 1 1)) (justify left))
+    (property "Intersheet References" "${INTERSHEET_REFS}" (id 0) (at 132.789 38.0375 0)
+      (effects (font (size 1 1)) (justify left) hide)
+    )
+  )
   (global_label "MOSI" (shape input) (at 44.196 183.642 0) (fields_autoplaced)
     (effects (font (size 1 1)) (justify left))
@@
     )
   )
-  (global_label "Col1" (shape input) (at 127.508 101.6 0) (fields_autoplaced)
-    (effects (font (size 1 1)) (justify left))
-    (property "Intersheet References" "${INTERSHEET_REFS}" (id 0) (at 132.789 101.5375 0)
-      (effects (font (size 1 1)) (justify left) hide)
-    )
-  )
-  (global_label "Col5" (shape input) (at 127.508 111.76 0) (fields_autoplaced)
+  (global_label "Col13" (shape input) (at 127.508 101.6 0) (fields_autoplaced)
+    (effects (font (size 1 1)) (justify left))
+    (property "Intersheet References" "${INTERSHEET_REFS}" (id 0) (at 133.7413 101.5375 0)
+      (effects (font (size 1 1)) (justify left) hide)
+    )
+  )
+  (global_label "Col9" (shape input) (at 127.508 111.76 0) (fields_autoplaced)
     (effects (font (size 1 1)) (justify left))
     (property "Intersheet References" "${INTERSHEET_REFS}" (id 0) (at 132.789 111.6975 0)
@@
     )
   )
-  (global_label "Col3" (shape input) (at 127.508 106.68 0) (fields_autoplaced)
-    (effects (font (size 1 1)) (justify left))
-    (property "Intersheet References" "${INTERSHEET_REFS}" (id 0) (at 132.789 106.6175 0)
+  (global_label "Col11" (shape input) (at 127.508 106.68 0) (fields_autoplaced)
+    (effects (font (size 1 1)) (justify left))
+    (property "Intersheet References" "${INTERSHEET_REFS}" (id 0) (at 133.7413 106.6175 0)
       (effects (font (size 1 1)) (justify left) hide)
     )
@@
     )
   )
-  (global_label "Col8" (shape input) (at 127.508 60.96 0) (fields_autoplaced)
+  (global_label "Col7" (shape input) (at 127.508 60.96 0) (fields_autoplaced)
     (effects (font (size 1 1)) (justify left))
     (property "Intersheet References" "${INTERSHEET_REFS}" (id 0) (at 132.789 60.8975 0)
@@
     )
     (path "/8d1ee0af-608f-46ba-ae0b-2302690e62f5/8467e55c-5ddd-477f-9ed0-4e68319a3a79"
-      (reference "K311") (unit 1) (value "KEYSW") (footprint "MX_Only:MXOnly-1U-Hotswap")
+      (reference "K312") (unit 1) (value "KEYSW") (footprint "MX_Only:MXOnly-1U-Hotswap")
     )
     (path "/8d1ee0af-608f-46ba-ae0b-2302690e62f5/4732cfd4-5bc1-48a5-bc98-3bdcdf99859e"
@@
     )
     (path "/8d1ee0af-608f-46ba-ae0b-2302690e62f5/32c567a9-f006-43e6-a74b-036e2419378d"
-      (reference "K411") (unit 1) (value "KEYSW") (footprint "MX_Only:MXOnly-1U-Hotswap")
+      (reference "K412") (unit 1) (value "KEYSW") (footprint "MX_Only:MXOnly-1U-Hotswap")
     )
     (path "/8d1ee0af-608f-46ba-ae0b-2302690e62f5/073b18b9-fe5c-4395-9748-d371957df215"

Commit message: Pull-up Resistors Added
Parts:
- added R8: 10k, Resistor_SMD:R_0402_1005Metric, symbol Device:R_Small
- added R9: 10K, Resistor_SMD:R_0402_1005Metric, symbol Device:R_Small
Connections:
- net Col2: no longer U1.12 (PB7)
- net SCL: now also R9.2
- net SDA: now also R8.2
- net VCC: now also R8.1, R9.1
- new net Col0: U1.12 (PB7)
Changed lines of the file:
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@@
   (junction (at 38.1 153.67) (diameter 0) (color 0 0 0 0)
   )
+  (junction (at 166.878 34.036) (diameter 0) (color 0 0 0 0)
+  )
+  (junction (at 163.83 42.926) (diameter 0) (color 0 0 0 0)
+  )
+  (junction (at 163.83 34.036) (diameter 0) (color 0 0 0 0)
+  )
   (junction (at 38.862 126.238) (diameter 0) (color 0 0 0 0)
   )
@@
   )
   (junction (at 41.656 128.778) (diameter 0) (color 0 0 0 0)
+  )
+  (junction (at 166.878 39.37) (diameter 0) (color 0 0 0 0)
   )
   (junction (at 30.226 75.184) (diameter 0) (color 0 0 0 0)
@@
     (stroke (width 0) (type default) (color 0 0 0 0))
   )
+  (wire (pts (xy 163.83 42.926) (xy 170.18 42.926))
+    (stroke (width 0) (type default) (color 0 0 0 0))
+  )
   (wire (pts (xy 44.6024 110.998) (xy 44.6024 116.078))
     (stroke (width 0) (type default) (color 0 0 0 0))
@@
     (stroke (width 0) (type default) (color 0 0 0 0))
   )
-  (wire (pts (xy 166.37 39.116) (xy 170.18 39.116))
+  (wire (pts (xy 166.878 34.036) (xy 163.83 34.036))
     (stroke (width 0) (type default) (color 0 0 0 0))
   )
@@
     (stroke (width 0) (type default) (color 0 0 0 0))
   )
+  (wire (pts (xy 169.164 36.576) (xy 170.18 36.576))
+    (stroke (width 0) (type default) (color 0 0 0 0))
+  )
   (wire (pts (xy 41.656 126.238) (xy 41.656 128.778))
     (stroke (width 0) (type default) (color 0 0 0 0))
@@
     (stroke (width 0) (type default) (color 0 0 0 0))
   )
-  (wire (pts (xy 166.37 36.576) (xy 170.18 36.576))
+  (wire (pts (xy 170.18 42.926) (xy 170.18 39.116))
+    (stroke (width 0) (type default) (color 0 0 0 0))
+  )
+  (wire (pts (xy 163.83 34.036) (xy 163.83 37.846))
     (stroke (width 0) (type default) (color 0 0 0 0))
   )
@@
     (stroke (width 0) (type default) (color 0 0 0 0))
   )
-  (wire (pts (xy 170.18 34.036) (xy 162.56 34.036))
+  (wire (pts (xy 170.18 34.036) (xy 166.878 34.036))
     (stroke (width 0) (type default) (color 0 0 0 0))
   )
@@
     (stroke (width 0) (type default) (color 0 0 0 0))
   )
+  (wire (pts (xy 163.83 34.036) (xy 162.56 34.036))
+    (stroke (width 0) (type default) (color 0 0 0 0))
+  )
   (wire (pts (xy 44.704 153.67) (xy 51.816 153.67))
     (stroke (width 0) (type default) (color 0 0 0 0))
@@
     (stroke (width 0) (type default) (color 0 0 0 0))
   )
+  (wire (pts (xy 162.052 42.926) (xy 163.83 42.926))
+    (stroke (width 0) (type default) (color 0 0 0 0))
+  )
   (wire (pts (xy 124.714 81.28) (xy 127.508 81.28))
     (stroke (width 0) (type default) (color 0 0 0 0))
@@
     (stroke (width 0) (type default) (color 0 0 0 0))
   )
+  (wire (pts (xy 166.878 34.036) (xy 166.878 34.29))
+    (stroke (width 0) (type default) (color 0 0 0 0))
+  )
   (wire (pts (xy 71.882 182.88) (xy 71.882 182.118))
     (stroke (width 0) (type default) (color 0 0 0 0))
@@
     (stroke (width 0) (type default) (color 0 0 0 0))
   )
+  (wire (pts (xy 162.052 39.37) (xy 166.878 39.37))
+    (stroke (width 0) (type default) (color 0 0 0 0))
+  )
   (wire (pts (xy 86.614 43.18) (xy 94.234 43.18))
     (stroke (width 0) (type default) (color 0 0 0 0))
@@
     (stroke (width 0) (type default) (color 0 0 0 0))
   )
+  (wire (pts (xy 166.878 39.37) (xy 169.164 39.37))
+    (stroke (width 0) (type default) (color 0 0 0 0))
+  )
   (wire (pts (xy 124.714 38.1) (xy 127.508 38.1))
     (stroke (width 0) (type default) (color 0 0 0 0))
@@
   )
   (wire (pts (xy 124.714 40.64) (xy 134.2136 40.64))
+    (stroke (width 0) (type default) (color 0 0 0 0))
+  )
+  (wire (pts (xy 169.164 39.37) (xy 169.164 36.576))
     (stroke (width 0) (type default) (color 0 0 0 0))
   )
@@
     )
   )
-  (global_label "SDA" (shape input) (at 166.37 39.116 180) (fields_autoplaced)
+  (global_label "SDA" (shape input) (at 162.052 42.926 180) (fields_autoplaced)
     (effects (font (size 1 1)) (justify right))
-    (property "Intersheet References" "${INTERSHEET_REFS}" (id 0) (at 161.6605 39.1785 0)
+    (property "Intersheet References" "${INTERSHEET_REFS}" (id 0) (at 157.3425 42.9885 0)
       (effects (font (size 1 1)) (justify right) hide)
     )
@@
     )
   )
-  (global_label "SCL" (shape input) (at 166.37 36.576 180) (fields_autoplaced)
+  (global_label "SCL" (shape input) (at 162.052 39.37 180) (fields_autoplaced)
     (effects (font (size 1 1)) (justify right))
-    (property "Intersheet References" "${INTERSHEET_REFS}" (id 0) (at 161.7081 36.6385 0)
+    (property "Intersheet References" "${INTERSHEET_REFS}" (id 0) (at 157.3901 39.4325 0)
       (effects (font (size 1 1)) (justify right) hide)
     )
@@
     )
   )
-  (global_label "Col2" (shape input) (at 127.508 55.88 0) (fields_autoplaced)
+  (global_label "Col0" (shape input) (at 127.508 55.88 0) (fields_autoplaced)
     (effects (font (size 1 1)) (justify left))
     (property "Intersheet References" "${INTERSHEET_REFS}" (id 0) (at 132.789 55.8175 0)
@@
     )
     (pin "1")
+  )
+  (symbol (lib_id "Device:R_Small") (at 166.878 36.83 0) (unit 1)
+    (in_bom yes) (on_board yes)
+    (property "Reference" "R9" (id 0) (at 163.83 35.56 0)
+      (effects (font (size 1.27 1.27)) (justify left))
+    )
+    (property "Value" "10K" (id 1) (at 166.878 38.608 90)
+      (effects (font (size 1.27 1.27)) (justify left))
+    )
+    (property "Footprint" "Resistor_SMD:R_0402_1005Metric" (id 2) (at 166.878 36.83 0)
+      (effects (font (size 1.27 1.27)) hide)
+    )
+    (property "Datasheet" "~" (id 3) (at 166.878 36.83 0)
+      (effects (font (size 1.27 1.27)) hide)
+    )
+    (pin "1")
+    (pin "2")
+  )
+  (symbol (lib_id "Device:R_Small") (at 163.83 40.386 0) (unit 1)
+    (in_bom yes) (on_board yes)
+    (property "Reference" "R8" (id 0) (at 161.29 37.592 0)
+      (effects (font (size 1.27 1.27)) (justify left))
+    )
+    (property "Value" "10k" (id 1) (at 163.83 41.91 90)
+      (effects (font (size 1.27 1.27)) (justify left))
+    )
+    (property "Footprint" "Resistor_SMD:R_0402_1005Metric" (id 2) (at 163.83 40.386 0)
+      (effects (font (size 1.27 1.27)) hide)
+    )
+    (property "Datasheet" "~" (id 3) (at 163.83 40.386 0)
+      (effects (font (size 1.27 1.27)) hide)
+    )
+    (pin "1")
+    (pin "2")
   )
   (symbol (lib_id "Device:C_Small") (at 22.098 71.882 0) (unit 1)
@@
       (reference "R7") (unit 1) (value "220") (footprint "Resistor_THT:R_Axial_DIN0204_L3.6mm_D1.6mm_P5.08mm_Horizontal")
     )
+    (path "/0d42412b-066b-493b-a941-af745b291ecb"
+      (reference "R8") (unit 1) (value "10k") (footprint "Resistor_SMD:R_0402_1005Metric")
+    )
+    (path "/0a8b2187-54b6-4d14-b24c-0bfa17f046b6"
+      (reference "R9") (unit 1) (value "10K") (footprint "Resistor_SMD:R_0402_1005Metric")
+    )
     (path "/ac780ebe-5afd-4e74-82f8-509da8ddaa4d"

Commit message: Ready for JLCPCB
Parts:
- added H1, H2, H3, H4: MountingHole, MountingHole:MountingHole_2.2mm_M2, symbol Mechanical:MountingHole
- C1, C2: value 20pF -> 12pF
- C3: footprint Capacitor_THT:C_Disc_D4.3mm_W1.9mm_P5.00mm -> Capacitor_SMD:C_0603_1608Metric
- R9: value 10K -> 10k
- Y1: value Crystal -> 16Mhz 9pF
Changed lines of the file:
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@@
     (pin "1")
+  )
+  (symbol (lib_id "Mechanical:MountingHole") (at 182.88 64.77 0) (unit 1)
+    (in_bom yes) (on_board yes) (fields_autoplaced)
+    (property "Reference" "H4" (id 0) (at 185.42 63.8615 0)
+      (effects (font (size 1.27 1.27)) (justify left))
+    )
+    (property "Value" "MountingHole" (id 1) (at 185.42 66.6366 0)
+      (effects (font (size 1.27 1.27)) (justify left))
+    )
+    (property "Footprint" "MountingHole:MountingHole_2.2mm_M2" (id 2) (at 182.88 64.77 0)
+      (effects (font (size 1.27 1.27)) hide)
+    )
+    (property "Datasheet" "~" (id 3) (at 182.88 64.77 0)
+      (effects (font (size 1.27 1.27)) hide)
+    )
   )
   (symbol (lib_id "Device:R_Small") (at 166.878 36.83 0) (unit 1)
@@
       (effects (font (size 1.27 1.27)) (justify left))
     )
-    (property "Value" "10K" (id 1) (at 166.878 38.608 90)
+    (property "Value" "10k" (id 1) (at 166.878 38.608 90)
       (effects (font (size 1.27 1.27)) (justify left))
     )
@@
       (effects (font (size 1.27 1.27)) (justify left))
     )
-    (property "Value" "20pF" (id 1) (at 16.256 73.66 0)
+    (property "Value" "12pF" (id 1) (at 16.256 73.66 0)
       (effects (font (size 1.27 1.27)) (justify left))
     )
@@
     (in_bom yes) (on_board yes)
     (property "Reference" "Y1" (id 0) (at 30.226 62.8101 0))
-    (property "Value" "Crystal" (id 1) (at 30.226 65.5852 0))
+    (property "Value" "16Mhz 9pF" (id 1) (at 30.226 65.5852 0))
     (property "Footprint" "Crystal:Crystal_SMD_3225-4Pin_3.2x2.5mm" (id 2) (at 30.226 69.342 0)
       (effects (font (size 1.27 1.27)) hide)
@@
     (pin "1")
   )
+  (symbol (lib_id "Mechanical:MountingHole") (at 162.56 64.262 0) (unit 1)
+    (in_bom yes) (on_board yes) (fields_autoplaced)
+    (property "Reference" "H1" (id 0) (at 165.1 63.3535 0)
+      (effects (font (size 1.27 1.27)) (justify left))
+    )
+    (property "Value" "MountingHole" (id 1) (at 165.1 66.1286 0)
+      (effects (font (size 1.27 1.27)) (justify left))
+    )
+    (property "Footprint" "MountingHole:MountingHole_2.2mm_M2" (id 2) (at 162.56 64.262 0)
+      (effects (font (size 1.27 1.27)) hide)
+    )
+    (property "Datasheet" "~" (id 3) (at 162.56 64.262 0)
+      (effects (font (size 1.27 1.27)) hide)
+    )
+  )
   (symbol (lib_id "Device:C_Small") (at 38.1 157.988 0) (unit 1)
     (in_bom yes) (on_board yes)
@@
       (effects (font (size 1.27 1.27)) (justify left))
     )
-    (property "Value" "20pF" (id 1) (at 39.6621 73.7549 0)
+    (property "Value" "12pF" (id 1) (at 39.6621 73.7549 0)
       (effects (font (size 1.27 1.27)) (justify left))
     )
@@
     (pin "1")
   )
+  (symbol (lib_id "Mechanical:MountingHole") (at 162.56 70.358 0) (unit 1)
+    (in_bom yes) (on_board yes) (fields_autoplaced)
+    (property "Reference" "H2" (id 0) (at 165.1 69.4495 0)
+      (effects (font (size 1.27 1.27)) (justify left))
+    )
+    (property "Value" "MountingHole" (id 1) (at 165.1 72.2246 0)
+      (effects (font (size 1.27 1.27)) (justify left))
+    )
+    (property "Footprint" "MountingHole:MountingHole_2.2mm_M2" (id 2) (at 162.56 70.358 0)
+      (effects (font (size 1.27 1.27)) hide)
+    )
+    (property "Datasheet" "~" (id 3) (at 162.56 70.358 0)
+      (effects (font (size 1.27 1.27)) hide)
+    )
+  )
   (symbol (lib_id "power:VCC") (at 47.498 100.076 0) (unit 1)
     (in_bom yes) (on_board yes) (fields_autoplaced)
@@
     (pin "2")
   )
+  (symbol (lib_id "Mechanical:MountingHole") (at 162.56 77.724 0) (unit 1)
+    (in_bom yes) (on_board yes) (fields_autoplaced)
+    (property "Reference" "H3" (id 0) (at 165.1 76.8155 0)
+      (effects (font (size 1.27 1.27)) (justify left))
+    )
+    (property "Value" "MountingHole" (id 1) (at 165.1 79.5906 0)
+      (effects (font (size 1.27 1.27)) (justify left))
+    )
+    (property "Footprint" "MountingHole:MountingHole_2.2mm_M2" (id 2) (at 162.56 77.724 0)
+      (effects (font (size 1.27 1.27)) hide)
+    )
+    (property "Datasheet" "~" (id 3) (at 162.56 77.724 0)
+      (effects (font (size 1.27 1.27)) hide)
+    )
+  )
   (symbol (lib_id "Device:C_Small") (at 21.844 158.242 0) (unit 1)
     (in_bom yes) (on_board yes)
@@
       (effects (font (size 1.27 1.27)) (justify left))
     )
-    (property "Footprint" "Capacitor_THT:C_Disc_D4.3mm_W1.9mm_P5.00mm" (id 2) (at 21.844 158.242 0)
+    (property "Footprint" "Capacitor_SMD:C_0603_1608Metric" (id 2) (at 21.844 158.242 0)
       (effects (font (size 1.27 1.27)) hide)
     )
@@
     )
     (path "/10822368-0e12-431b-8c12-cb7f4bbe9740"
-      (reference "C1") (unit 1) (value "20pF") (footprint "Capacitor_SMD:C_0402_1005Metric")
+      (reference "C1") (unit 1) (value "12pF") (footprint "Capacitor_SMD:C_0402_1005Metric")
     )
     (path "/4928f433-c898-4679-bfab-69ab45c14c50"
-      (reference "C2") (unit 1) (value "20pF") (footprint "Capacitor_SMD:C_0402_1005Metric")
+      (reference "C2") (unit 1) (value "12pF") (footprint "Capacitor_SMD:C_0402_1005Metric")
     )
     (path "/d860e7b5-f373-48d8-99d4-2dc054110bb6"
-      (reference "C3") (unit 1) (value "4.7uF") (footprint "Capacitor_THT:C_Disc_D4.3mm_W1.9mm_P5.00mm")
+      (reference "C3") (unit 1) (value "4.7uF") (footprint "Capacitor_SMD:C_0603_1608Metric")
     )
     (path "/f77aa4d6-9493-44e2-970c-08355ba7fdf3"
@@
       (reference "D64") (unit 1) (value "LED") (footprint "LED_THT:LED_D3.0mm_Clear")
     )
+    (path "/434f2fbd-322f-4975-a8ae-f9d4f20db4f8"
+      (reference "H1") (unit 1) (value "MountingHole") (footprint "MountingHole:MountingHole_2.2mm_M2")
+    )
+    (path "/7f455d34-a63c-487b-93fa-01047082e5b8"
+      (reference "H2") (unit 1) (value "MountingHole") (footprint "MountingHole:MountingHole_2.2mm_M2")
+    )
+    (path "/d2bad25d-18ac-4ba7-a263-80bcc919065f"
+      (reference "H3") (unit 1) (value "MountingHole") (footprint "MountingHole:MountingHole_2.2mm_M2")
+    )
+    (path "/0366b911-fa8d-4547-9c08-21d6047f71ba"
+      (reference "H4") (unit 1) (value "MountingHole") (footprint "MountingHole:MountingHole_2.2mm_M2")
+    )
     (path "/51a3cb30-7fac-47df-8e5e-a5ae1a15d9b8"
       (reference "J1") (unit 1) (value "ICSP") (footprint "Connector_PinHeader_2.54mm:PinHeader_2x03_P2.54mm_Vertical")
@@
     )
     (path "/0a8b2187-54b6-4d14-b24c-0bfa17f046b6"
-      (reference "R9") (unit 1) (value "10K") (footprint "Resistor_SMD:R_0402_1005Metric")
+      (reference "R9") (unit 1) (value "10k") (footprint "Resistor_SMD:R_0402_1005Metric")
     )
     (path "/ac780ebe-5afd-4e74-82f8-509da8ddaa4d"
@@
     )
     (path "/16eae8dc-1dc8-472c-8458-29d80b10b0b3"
-      (reference "Y1") (unit 1) (value "Crystal") (footprint "Crystal:Crystal_SMD_3225-4Pin_3.2x2.5mm")
-    )
-  )
+      (reference "Y1") (unit 1) (value "16Mhz 9pF") (footprint "Crystal:Crystal_SMD_3225-4Pin_3.2x2.5mm")
+    )
+  )
